File: kicad/shoedler54.kicad_pcb (KiCad board)
At the start: 2 copper layers, 141.5 x 124.7 mm, 63 parts

Commit message: Fixes PCB silkscreen text, as JLCPCB fears having ergogen.xyz on it will trouble the customs paw patrol. Also made GND fill zones better by adding some vias.
Routing:
- net GND: vias 2 -> 21
Other:
- board text added: "(contains many declarations)"
- board text removed: "made with ergogen.xyz"
